File: LoopEcho.kicad_sch (KiCad schematic)
At the start: 77 parts, among them J1 9V / GND, J2 IN / OUT / GND, J3 INSERT (TRS), U1 PT2399, U2 TL072, U3 TL072, U4 TL072, U5 78L05

Commit message: v1.0 SMD schematic: SEND / switched RETURN, TONE on every repeat, LFO into the TIME / 2k7 node, AMS1117, JLC parts; v0.1 generator kept
Co-Authored-By: Claude Opus 5.5 <noreply@anthropic.com>
Parts:
- removed C1: 100u, symbol Device:C_Polarized
- removed C11, C23, C26, C28, C5, C9: 10u, symbol Device:C_Polarized
- removed C12, C7: 47u, symbol Device:C_Polarized
- removed C30: 4u7, symbol Device:C_Polarized
- removed D1: 1N5817, symbol Device:D_Schottky
- removed D2, D3: 1N4148, symbol Device:D
- removed J1: 9V / GND, symbol Connector_Generic:Conn_01x02
- removed J2: IN / OUT / GND, symbol Connector_Generic:Conn_01x03
- removed J3: INSERT (TRS), symbol Connector_Audio:AudioJack3_SwitchTR
- removed U4: TL072, symbol Amplifier_Operational:TL072
- removed U5: 78L05, symbol Regulator_Linear:L78L05_TO92
- added C1: 22u, Capacitor_SMD:C_0805_2012Metric_Pad1.18x1.45mm_HandSolder, symbol Device:C
- added C11, C28, C34, C7: 10u, Capacitor_SMD:C_0805_2012Metric_Pad1.18x1.45mm_HandSolder, symbol Device:C
- added C12: 1n, Capacitor_SMD:C_0805_2012Metric_Pad1.18x1.45mm_HandSolder, symbol Device:C
- added C23, C30: 10n, Capacitor_SMD:C_0805_2012Metric_Pad1.18x1.45mm_HandSolder, symbol Device:C
- added C26: 47n, Capacitor_SMD:C_0805_2012Metric_Pad1.18x1.45mm_HandSolder, symbol Device:C
- added C32: 1u, Capacitor_SMD:C_0805_2012Metric_Pad1.18x1.45mm_HandSolder, symbol Device:C
- added C33: 4u7, Capacitor_SMD:C_0805_2012Metric_Pad1.18x1.45mm_HandSolder, symbol Device:C
- added C5: 100n, Capacitor_SMD:C_0805_2012Metric_Pad1.18x1.45mm_HandSolder, symbol Device:C
- added C9: 47u, Capacitor_SMD:C_1206_3216Metric_Pad1.33x1.80mm_HandSolder, symbol Device:C
- added D1: SS14, Diode_SMD:D_SMA, symbol Diode:SS14
- added D2, D3: 1N4148W, Diode_SMD:D_SOD-123, symbol Diode:1N4148W
- added D6: LED, LED_THT:LED_D3.0mm, symbol Device:LED
- added J1: IN/LED/GND/OUT, Connector_PinHeader_2.54mm:PinHeader_1x04_P2.54mm_Vertical, symbol Connector_Generic:Conn_01x04
- added J1: 9V, Connector_Wire:SolderWire-0.5sqmm_1x01_D0.9mm_OD2.1mm, symbol Connector_Generic:Conn_01x01
- added J2: G, Connector_Wire:SolderWire-0.5sqmm_1x01_D0.9mm_OD2.1mm, symbol Connector_Generic:Conn_01x01
- added J2: IG, Connector_Wire:SolderWire-0.5sqmm_1x01_D0.9mm_OD2.1mm, symbol Connector_Generic:Conn_01x01
- added J3: OG, Connector_Wire:SolderWire-0.5sqmm_1x01_D0.9mm_OD2.1mm, symbol Connector_Generic:Conn_01x01
- added J4: SEND, Connector_Wire:SolderWire-0.5sqmm_1x01_D0.9mm_OD2.1mm, symbol Connector_Generic:Conn_01x01
- added J5: SG, Connector_Wire:SolderWire-0.5sqmm_1x01_D0.9mm_OD2.1mm, symbol Connector_Generic:Conn_01x01
- added J6: RET, Connector_Wire:SolderWire-0.5sqmm_1x01_D0.9mm_OD2.1mm, symbol Connector_Generic:Conn_01x01
- added J7: RETN, Connector_Wire:SolderWire-0.5sqmm_1x01_D0.9mm_OD2.1mm, symbol Connector_Generic:Conn_01x01
- added J8: RG, Connector_Wire:SolderWire-0.5sqmm_1x01_D0.9mm_OD2.1mm, symbol Connector_Generic:Conn_01x01
- added R31: 22k, Resistor_SMD:R_0805_2012Metric_Pad1.20x1.40mm_HandSolder, symbol Device:R
- added R32: 33k, Resistor_SMD:R_0805_2012Metric_Pad1.20x1.40mm_HandSolder, symbol Device:R
- added RV6: B100k, Potentiometer_THT:Potentiometer_Alpha_RD901F-40-00D_Single_Vertical, symbol Device:R_Potentiometer
- added U4: LM358, Package_SO:SOIC-8_3.9x4.9mm_P1.27mm, symbol Amplifier_Operational:LM358
- added U5: AMS1117-5.0, Package_TO_SOT_SMD:SOT-223-3_TabPin2, symbol Regulator_Linear:AMS1117-5.0
- C10: value 1n -> 100n; footprint (none) -> Capacitor_SMD:C_0805_2012Metric_Pad1.18x1.45mm_HandSolder; LCSC (none) -> C49678
- C13, C6: value 100n -> 10u; footprint (none) -> Capacitor_SMD:C_0805_2012Metric_Pad1.18x1.45mm_HandSolder; LCSC (none) -> C15850
- C14: value 100n -> 47u; footprint (none) -> Capacitor_SMD:C_1206_3216Metric_Pad1.33x1.80mm_HandSolder; LCSC (none) -> C96123
- C15, C16, C3, C4, C8: footprint (none) -> Capacitor_SMD:C_0805_2012Metric_Pad1.18x1.45mm_HandSolder; LCSC (none) -> C49678
- C17, C22: value 2n2 -> 100n; footprint (none) -> Capacitor_SMD:C_0805_2012Metric_Pad1.18x1.45mm_HandSolder; LCSC (none) -> C49678
- C18, C21: value 10n -> 100n; footprint (none) -> Capacitor_SMD:C_0805_2012Metric_Pad1.18x1.45mm_HandSolder; LCSC (none) -> C49678
- C19: value 100n -> 2n2; footprint (none) -> Capacitor_SMD:C_0805_2012Metric_Pad1.18x1.45mm_HandSolder; LCSC (none) -> C28260
- C2: value 100n -> 22u; footprint (none) -> Capacitor_SMD:C_0805_2012Metric_Pad1.18x1.45mm_HandSolder; LCSC (none) -> C45783
- C20: value 100n -> 10n; footprint (none) -> Capacitor_SMD:C_0805_2012Metric_Pad1.18x1.45mm_HandSolder; LCSC (none) -> C1710
- C24: value 47n -> 2n2; footprint (none) -> Capacitor_SMD:C_0805_2012Metric_Pad1.18x1.45mm_HandSolder; LCSC (none) -> C28260
- C25, C31: value 1u -> 10u; footprint (none) -> Capacitor_SMD:C_0805_2012Metric_Pad1.18x1.45mm_HandSolder; LCSC (none) -> C15850
- C27, C29: footprint (none) -> Capacitor_SMD:C_0805_2012Metric_Pad1.18x1.45mm_HandSolder; LCSC (none) -> C28323
- R1, R12, R14, R15, R16, R17, R18, R2, R7, R8: footprint (none) -> Resistor_SMD:R_0805_2012Metric_Pad1.20x1.40mm_HandSolder; LCSC (none) -> C17414
- R10: value 100k -> 100; footprint (none) -> Resistor_SMD:R_0805_2012Metric_Pad1.20x1.40mm_HandSolder; LCSC (none) -> C17408
- R11: value 1k -> 100k; footprint (none) -> Resistor_SMD:R_0805_2012Metric_Pad1.20x1.40mm_HandSolder; LCSC (none) -> C149504
- R13: footprint (none) -> Resistor_SMD:R_0805_2012Metric_Pad1.20x1.40mm_HandSolder; LCSC (none) -> C17475
- R19: footprint (none) -> Resistor_SMD:R_0805_2012Metric_Pad1.20x1.40mm_HandSolder; LCSC (none) -> C17513
- R20: value 1k -> 2k7; footprint (none) -> Resistor_SMD:R_0805_2012Metric_Pad1.20x1.40mm_HandSolder; LCSC (none) -> C17530
- R21: value 1M -> 1k; footprint (none) -> Resistor_SMD:R_0805_2012Metric_Pad1.20x1.40mm_HandSolder; LCSC (none) -> C17513
- R22: value 1k -> 1M; footprint (none) -> Resistor_SMD:R_0805_2012Metric_Pad1.20x1.40mm_HandSolder; LCSC (none) -> C17514
- R23: value 100k -> 1k; footprint (none) -> Resistor_SMD:R_0805_2012Metric_Pad1.20x1.40mm_HandSolder; LCSC (none) -> C17513
- R24: value 1M -> 100k; footprint (none) -> Resistor_SMD:R_0805_2012Metric_Pad1.20x1.40mm_HandSolder; LCSC (none) -> C149504
- R25: footprint (none) -> Resistor_SMD:R_0805_2012Metric_Pad1.20x1.40mm_HandSolder; LCSC (none) -> C17514
- R26: value 1k -> 2k2; footprint (none) -> Resistor_SMD:R_0805_2012Metric_Pad1.20x1.40mm_HandSolder; LCSC (none) -> C17520
- R27: value 47k -> 1M; footprint (none) -> Resistor_SMD:R_0805_2012Metric_Pad1.20x1.40mm_HandSolder; LCSC (none) -> C17514
- R28: value 10k -> 1k; footprint (none) -> Resistor_SMD:R_0805_2012Metric_Pad1.20x1.40mm_HandSolder; LCSC (none) -> C17513
- R29: value 22k -> 47k; footprint (none) -> Resistor_SMD:R_0805_2012Metric_Pad1.20x1.40mm_HandSolder; LCSC (none) -> C17713
- R3: value 1M -> 4k7; footprint (none) -> Resistor_SMD:R_0805_2012Metric_Pad1.20x1.40mm_HandSolder; LCSC (none) -> C17673
- R30: value 100k -> 10k; footprint (none) -> Resistor_SMD:R_0805_2012Metric_Pad1.20x1.40mm_HandSolder; LCSC (none) -> C17414
- R4: value 100 -> 1M; footprint (none) -> Resistor_SMD:R_0805_2012Metric_Pad1.20x1.40mm_HandSolder; LCSC (none) -> C17514
- R5: value 1M -> 100; footprint (none) -> Resistor_SMD:R_0805_2012Metric_Pad1.20x1.40mm_HandSolder; LCSC (none) -> C17408
- R6: value 10k -> 1M; footprint (none) -> Resistor_SMD:R_0805_2012Metric_Pad1.20x1.40mm_HandSolder; LCSC (none) -> C17514
- R9: value 100 -> 10k; footprint (none) -> Resistor_SMD:R_0805_2012Metric_Pad1.20x1.40mm_HandSolder; LCSC (none) -> C17414
- RV1, RV2: footprint (none) -> Potentiometer_THT:Potentiometer_Alpha_RD901F-40-00D_Single_Vertical; now left out of the parts list
- RV3: value B10k -> B50k; footprint (none) -> Potentiometer_THT:Potentiometer_Alpha_RD901F-40-00D_Single_Vertical; Panel REPEAT -> TONE; now left out of the parts list
- RV4: value B1M -> B10k; footprint (none) -> Potentiometer_THT:Potentiometer_Alpha_RD901F-40-00D_Single_Vertical; Panel RATE -> REPEAT; now left out of the parts list
- RV5: value B100k -> B1M; footprint (none) -> Potentiometer_THT:Potentiometer_Alpha_RD901F-40-00D_Single_Vertical; Panel DEPTH -> RATE; now left out of the parts list
- U1: footprint (none) -> Package_SO:SOIC-16_3.9x9.9mm_P1.27mm; LCSC (none) -> C126407
- U2, U3: footprint (none) -> Package_SO:SOIC-8_3.9x4.9mm_P1.27mm; FT Rotation Offset (none) -> 270; LCSC (none) -> C6961
Connections:
- net +5V: now also C8.1, C7.1, U5.2 (VO); no longer C6.1
- net +9V: now also C6.1, R3.1, C1.1, C5.1, D1.1 (K), U4.8 (V+), U5.3 (VI)
- net DIN: now also C20.1; no longer C18.1
- net DRY: now also C21.1, R7.1; no longer C19.1, R6.1
- net GND: now also C15.2, C16.2, C20.2, C8.2, R20.2, R25.2, R4.2, RV4.1, C1.2, C23.2, C26.2, C30.2, C5.2, C7.2, C9.2, D2.1 (K), D3.2 (A), J1.3 (Pin_3), J2.1 (Pin_1), J2.1 (Pin_1), J3.1 (Pin_1), J5.1 (Pin_1), J8.1 (Pin_1), RV6.1, U4.4 (V-), U5.1 (GND); no longer C13.2, C18.2, C21.2, C24.2, R10.2, R23.2, R3.2, RV3.1, RV5.1
- net IN: now also C10.1, R4.1, J1.1 (Pin_1); no longer C8.1, R3.1
- net LP1I: now also C19.1; no longer C17.1
- net LP1O: now also C19.2; no longer C17.2
- net LP2I: now also C24.1; no longer C22.1
- net LP2O: now also C24.2, C25.1; no longer C22.2
- net MIXW: now also C11.1
- net OP1I: now also C17.1; no longer C15.1
- net OP1O: now also C17.2; no longer C15.2
- net OP2I: now also C18.1; no longer C16.1
- net OP2O: now also C18.2; no longer C16.2
- net OUT: now also C13.2, R11.1, J1.4 (Pin_4); no longer R10.1
- net RET: now also C29.1, R25.1, J6.1 (Pin_1); no longer C27.1, R24.1
- net RPT: now also C22.1, RV4.2; no longer C20.1, RV3.2
- net SEND: now also R23.2, R24.1, J4.1 (Pin_1), J7.1 (Pin_1); no longer R22.2, R23.1
- net SQR: now also RV5.2, RV5.3, R31.2, U4.7; no longer R29.2, RV4.2, RV4.3
- net TRI: now also R30.1, C32.2, C33.1, U4.1; no longer C29.2, R28.1
- net VB: now also R22.2, R27.2, R6.2, C9.1, U4.3 (+), U4.6 (-); no longer R21.2, R25.2, R5.2
- net VCO: no longer C31.2
- net W: now also C27.1, R21.1; no longer C25.1, R20.1
- net at R15.1: now also C22.2; no longer C20.2
- net at R28.2: now also RV4.3, D2.2 (A), D3.1 (K); no longer R29.1
- net at U3.1, U3.2 (-): now also C28.1
- net at R22.1: now also C27.2, U3.3 (+)
- net TMIN: now reaches RV1.2, RV1.3
- net TMIN: now also R20.1, C34.2; no longer R11.1
- net at U1.2 (REF): now also C14.1
- net at R8.2, R9.1: now also R7.2, U2.6 (-), C12.1; no longer C10.2, U2.7
- net at R16.2, R17.1, R18.1: now also C23.1; no longer C21.1
- net at R26.2: now also R27.1, U3.5 (+), C30.1; no longer RV3.3
- net at C13.1: now also R10.2; no longer U1.7 (CC1)
- net at R19.1: now also C25.2
- net at U3.6 (-), U3.7: now also C31.1
- net at R26.1: now also RV3.2, RV3.3
- net at R30.2: now also R31.1, U4.5 (+); no longer C31.1
- net at R9.2: now also R10.1, U2.7, C12.2
- net at R14.1: now also C21.2; no longer C19.2
- net at U1.8 (CC0): now also C16.1; no longer C14.1
- new net: D6.2 (A), R3.2
- new net: C26.1, R21.2, RV2.3
- new net: C28.2, R23.1
- new net: C32.1, R29.2, U4.2 (-)
- new net: R32.1, RV6.2
- new net: C33.2, RV6.3
- new net: C15.1, U1.7 (CC1)
- new net: R29.1, RV5.1
- new net: C31.2, R28.1
- new net: C11.2, R8.1
- new net: R5.2, R6.1, U2.3 (+)
- new net: C29.2, RV3.1
- new net: D1.2 (A), J1.1 (Pin_1)
- new net: C10.2, R5.1
- new net: C34.1, R32.2
- new net LED_K: D6.1 (K), J1.2 (Pin_2)
- no-connect marks 2 -> 1
Other:
- note added: "A fuzz in the loop adds gain every pass: the 1N4148W pair caps the loop at about +-0.6 V."
- note added: "DELAY: PT2399 (U1), Small Time network. TIME = B50k + 2k7 (VCO to ground); the LFO enters at TMIN"
- note added: "FEEDBACK LOOP: SEND (U3A) -> loop -> RETURN (no plug = internal) -> TONE -> U3B -> limiter -> REPEAT"
- note added: "MODULATION: LFO (U4, LM358) -> DEPTH -> 33k + 10u -> TMIN (even depth across TIME). ~0.5-12 Hz"
- note added: "No plug in RETURN: the jack's switch ties RET to SEND (internal path). TONE acts on every repeat in both cases."
- note added: "POWER (SS14, AMS1117-5.0 for the PT2399), VB, STATUS LED, FOOTSWITCH HEADER, JACK PADS"
- note removed: "A fuzz in the loop adds gain every pass: the 1N4148s cap the loop at about +-0.6 V so oscillation stays musical."
- note removed: "DELAY: PT2399 (U1), network as Small Time. TIME = R11 1k + B50k (VCO to ground)"
- note removed: "FEEDBACK LOOP: SEND (U3A) -> TRS insert -> RETURN (U3B) -> limiter -> REPEAT. No plug: ring-normal ties RETURN to SEND"
- note removed: "MODULATION: LFO (U4) -> DEPTH -> VCO pin (wow / chorus on the echoes). ~0.5-12 Hz"
- note removed: "Only the repeats circulate: the first echo is clean, each later echo goes through the loop again."
- note removed: "POWER: 9 V, VB 4.5 V for the TL072s, 5 V regulator for the PT2399"
- note removed: "The LFO current into pin 6 swings the clock: about +-15 uA at full DEPTH. Compare with the mod examples."
- title: Loop Echo (breadboard) -> Loop Echo

Commit message: v1.0 board: 1590BB landscape, all five jacks on top (OUT RETURN DC SEND IN)
- Schematic: board-mounted PJ-646F jacks (RETURN tip switch = SEND), A-4118 DC jack
  (centre negative, pads 2 + 3 to the SS14), 1x6 header in the SwitchPCB v2 order;
  wire pads removed. ERC 0.
- Footprints from the Tayda drawings in SuperFreq.pretty.
- Board: 100.0 x 83.5 mm, lid-boss cut-outs, footswitch notch, pots 2x3 + LED on the
  back, J1 vertical beside the notch (user). Routed: DRC 0 errors / 0 unconnected,
  parity clean, 63 vias. Board is hand-edited now: don't re-run buildpcb_loopecho.py.

Co-Authored-By: Claude Opus 5.5 <noreply@anthropic.com>
Parts:
- removed J1: IN/LED/GND/OUT, Connector_PinHeader_2.54mm:PinHeader_1x04_P2.54mm_Vertical, symbol Connector_Generic:Conn_01x04
- removed J1: 9V, Connector_Wire:SolderWire-0.5sqmm_1x01_D0.9mm_OD2.1mm, symbol Connector_Generic:Conn_01x01
- removed J2: G, Connector_Wire:SolderWire-0.5sqmm_1x01_D0.9mm_OD2.1mm, symbol Connector_Generic:Conn_01x01
- removed J2: IG, Connector_Wire:SolderWire-0.5sqmm_1x01_D0.9mm_OD2.1mm, symbol Connector_Generic:Conn_01x01
- removed J3: OG, Connector_Wire:SolderWire-0.5sqmm_1x01_D0.9mm_OD2.1mm, symbol Connector_Generic:Conn_01x01
- removed J4: SEND, Connector_Wire:SolderWire-0.5sqmm_1x01_D0.9mm_OD2.1mm, symbol Connector_Generic:Conn_01x01
- removed J5: SG, Connector_Wire:SolderWire-0.5sqmm_1x01_D0.9mm_OD2.1mm, symbol Connector_Generic:Conn_01x01
- removed J6: RET, Connector_Wire:SolderWire-0.5sqmm_1x01_D0.9mm_OD2.1mm, symbol Connector_Generic:Conn_01x01
- removed J7: RETN, Connector_Wire:SolderWire-0.5sqmm_1x01_D0.9mm_OD2.1mm, symbol Connector_Generic:Conn_01x01
- removed J8: RG, Connector_Wire:SolderWire-0.5sqmm_1x01_D0.9mm_OD2.1mm, symbol Connector_Generic:Conn_01x01
- added J1: IJ/IN/LED/GND/OUT/OJ, Connector_PinHeader_2.54mm:PinHeader_1x06_P2.54mm_Vertical, symbol Connector_Generic:Conn_01x06
- added J2: INPUT, SuperFreq:Jack_6.35mm_PJ-646F_Horizontal, symbol Connector_Audio:AudioJack3_Switch
- added J3: OUTPUT, SuperFreq:Jack_6.35mm_PJ-646F_Horizontal, symbol Connector_Audio:AudioJack3_Switch
- added J4: SEND, SuperFreq:Jack_6.35mm_PJ-646F_Horizontal, symbol Connector_Audio:AudioJack3_Switch
- added J5: RETURN, SuperFreq:Jack_6.35mm_PJ-646F_Horizontal, symbol Connector_Audio:AudioJack3_Switch
- added J6: DC 9V, SuperFreq:DC_Jack_2.1mm_A-4118_Horizontal, symbol Connector:Barrel_Jack_Switch
Connections:
- net GND: now also J1.4 (Pin_4), J2.S, J3.S, J4.S, J5.S, J6.1
- net IN: now also J1.2 (Pin_2)
- net LED_K: now also J1.3 (Pin_3)
- net OUT: now also J1.5 (Pin_5)
- net RET: now also J5.T
- net SEND: now also J4.T, J5.TN
- net at D1.2 (A): now also J6.2, J6.3
- new net IJ: J1.1 (Pin_1), J2.T
- new net OJ: J1.6 (Pin_6), J3.T
- no-connect marks 1 -> 16
Other:
- note added: "POWER (SS14, AMS1117-5.0 for the PT2399), VB, STATUS LED, FOOTSWITCH HEADER, JACKS"
- note removed: "POWER (SS14, AMS1117-5.0 for the PT2399), VB, STATUS LED, FOOTSWITCH HEADER, JACK PADS"

Commit message: Two footswitches: LOOP (left) switches the effects loop, BYPASS (right)
- Schematic: J7 header for a second SwitchPCB v2 wired as a loop selector
  (IJ = SEND, IN = SEND jack, LED = LOOP LED D7 / R33, OUT = RETURN jack, OJ = RET).
  Loop off: RET = SEND and the SEND jack is grounded. ERC 0.
- Board (hand-edited, reworked in place): second notch, both headers beside their
  notches like the user's J1, LEDs at X +-28 / Y -14.2, U1 / U2 / U4 groups
  re-placed, re-routed: DRC 0 errors / 0 unconnected, parity clean, 47 vias.
- buildpcb_loopecho.py marked out of date.

Co-Authored-By: Claude Opus 5.5 <noreply@anthropic.com>
Parts:
- added D7: LED, LED_THT:LED_D3.0mm, symbol Device:LED
- added J7: LOOP SW, Connector_PinHeader_2.54mm:PinHeader_1x06_P2.54mm_Vertical, symbol Connector_Generic:Conn_01x06
- added R33: 4k7, Resistor_SMD:R_0805_2012Metric_Pad1.20x1.40mm_HandSolder, symbol Device:R
Connections:
- net +9V: now also R33.1
- net GND: now also J7.4 (Pin_4)
- net RET: now also J7.6 (Pin_6); no longer J5.T
- net SEND: now also J7.1 (Pin_1); no longer J4.T
- new net: D7.2 (A), R33.2
- new net LED2_K: D7.1 (K), J7.3 (Pin_3)
- new net RETJ: J5.T, J7.5 (Pin_5)
- new net SENDJ: J4.T, J7.2 (Pin_2)
Other:
- note added: "LOOP FOOTSWITCH (2nd SwitchPCB v2): RET = SEND or RETURN"
- note added: "LOOP footswitch off: RET = SEND (internal path), SEND jack grounded. On: RET = RETURN jack; no plug in RETURN = its switch ties it to SEND. TONE acts on every repeat in all cases."
- note added: "SwitchPCB pads: OJ = OUT when engaged, IJ when bypassed; IN = IJ when engaged, GND when bypassed; LED to GND when engaged."
- note removed: "No plug in RETURN: the jack's switch ties RET to SEND (internal path). TONE acts on every repeat in both cases."
